File: PCB/RFlyOne.kicad_sch (KiCad schematic)
At the start: 168 parts, among them J1 UFL, J2 UFL, Q1 AO3401A, Q2 AO3401A, SW1 TS24CA, SW2 TS24CA, SW4 TS24CA, SW5 TS24CA, U1 TQP3M9036, U10 ATGM332D-5N31, U11 ESP32_S3_MINI, U12 E80-900M2212S, U13 RT9193-33GB, U14 RT8097CHGE, U15 BMI270, U16 MMC5983MA, U17 BQ25606RGER, U18 TPS61023DRLR, U19 CH32V003F4U6, U2 TLV3201, U20 TXU0202DTTR, U21 TPS7A0230-3V0, U22 240x320_2.4in_TFT, U3 TA0970A, U4 TQP3M9036, U5 TA0970A, U6 AD8313ARMZ, U7 RP2040, U8 W25Q128, U9 12MHz

Commit message: checkpoint
Parts:
- added C64, C65, C66: 0.1uF, Capacitor_SMD:C_0402_1005Metric, symbol Device:C_Small
- TP4: value BOOT -> RP_BOOT
Connections:
- net +D3V3: now also C64.1, C65.1, C66.1
- net BATT_ADC: now also U11.10 (IO6)
- net CH32_RX: now also U19.20 (PD6)
- net CH32_TX: now also U19.19 (PD5)
- net CHARGE: now also U19.9 (PC2)
- net CONN_RP_USB_DN: now also D2.1; no longer D2.3
- net CONN_RP_USB_DP: now also D2.3; no longer D2.1
- net GND: now also C64.2, C65.2, C66.2
- net LEFT_BTN: now also U19.16 (PD2)
- net LORA_BUSY: now also U11.20 (IO16); no longer U11.10 (IO6)
- net OK_BTN: now also U19.17 (PD3)
- net PG: now also U19.10 (PC3)
- net PPS: now also U11.21 (IO17); no longer U11.20 (IO16)
- net RIGHT_BTN: now also U19.18 (PD4)
- net RP_USB_DN: now also D2.6; no longer D2.4
- net RP_USB_DP: now also D2.4; no longer D2.6
- net SPI_CS: now also R12.1, R16.2, U8.1 (~{CS}); no longer R16.1
- net BTMGR_ESP32_RX renamed CONV_CH32_TX
- net BTMGR_ESP32_TX renamed CONV_CH32_RX
- new net: R16.1, TP4.1
- no-connect marks 82 -> 83
Other:
- moved on the sheet: D4, R33, R34, TP4, TP9

Commit message: checkpoint
Parts:
- added TP12: D3V3, easyeda2kicad:TestPoint, symbol Connector:TestPoint
- added TP13: 3V3, easyeda2kicad:TestPoint, symbol Connector:TestPoint
- added TP14: 5V, easyeda2kicad:TestPoint, symbol Connector:TestPoint
- added TP15: 5VU, easyeda2kicad:TestPoint, symbol Connector:TestPoint
- added TP16: SDA, easyeda2kicad:TestPoint, symbol Connector:TestPoint
- added TP17: SCL, easyeda2kicad:TestPoint, symbol Connector:TestPoint
- added TP18: CHARGE, easyeda2kicad:TestPoint, symbol Connector:TestPoint
- added TP19: PG, easyeda2kicad:TestPoint, symbol Connector:TestPoint
- added TP20: PULSE, easyeda2kicad:TestPoint, symbol Connector:TestPoint
Connections:
- net +3V3: now also TP13.1
- net +5V: now also TP14.1
- net +5VU: now also TP15.1
- net +D3V3: now also TP12.1
- net CHARGE: now also TP18.1
- net PG: now also TP19.1
- net PULSE: now also TP20.1
- net SCL: now also TP17.1
- net SDA: now also TP16.1

Commit message: checkpoint
Parts:
- added JP2: PWRBYPASS, Jumper:SolderJumper-2_P1.3mm_Open_RoundedPad1.0x1.5mm, symbol Jumper:SolderJumper_2_Open
- added R47: 5.1k, Resistor_SMD:R_0402_1005Metric, symbol Device:R_Small
- added TP21: CH32_TX, easyeda2kicad:TestPoint, symbol Connector:TestPoint
- added TP22: CH32_RX, easyeda2kicad:TestPoint, symbol Connector:TestPoint
- D4: footprint (none) -> easyeda2kicad:LED-SMD_L1.6-W1.1-R-RD_WHITE
- JP1: footprint (none) -> Jumper:SolderJumper-2_P1.3mm_Open_RoundedPad1.0x1.5mm
- TP5: value UART_TX -> RP_TX
- TP6: value UART_RX -> RP_RX
Connections:
- net CONV_CH32_RX: now also U11.22 (IO18), TP22.1
- net CONV_CH32_TX: now also U11.25 (IO21), TP21.1
- net GND: now also D4.1 (K), JP2.2 (B)
- net PULSE: now also U7.27 (GPIO16)
- net PWR_BTN: now also U19.5 (PD0)
- net RP2040_RX: now also TP8.1, U11.30 (IO48), U7.7 (GPIO5)
- net RP2040_TX: now also TP7.1, U11.27 (IO47), U7.6 (GPIO4)
- net at Q2.1 (G), R32.1, R33.1: now also JP2.1 (A)
- net at U7.2 (GPIO0): now also TP5.1
- net at U7.3 (GPIO1): now also TP6.1
- net at U19.2 (PA1): now also R47.1
- net at D4.2 (A): now also R47.2
- no-connect marks 83 -> 79
Other:
- note removed: "Temporarily Unconnected"
- moved on the sheet: C54, D4, TP1, TP5, TP6, TP7, TP8

Commit message: checkpoint
Parts:
- BT1: footprint (none) -> easyeda2kicad:Battery
Connections:
- net at U7.28 (GPIO17): now also TP1.1
Other:
- moved on the sheet: TP1
Changed lines of the file:
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@@
 	(wire
 		(pts
+			(xy 414.02 290.83) (xy 408.94 290.83)
+		)
+		(stroke
+			(width 0)
+			(type default)
+		)
+	)
+	(wire
+		(pts
 			(xy 224.79 299.72) (xy 224.79 304.8)
 		)
@@
 	(global_label "BIAS_TEE_EN"
 		(shape input)
-		(at 433.07 318.77 0)
+		(at 414.02 299.72 0)
 		(fields_autoplaced yes)
 		(effects
@@
 		)
 		(property "Intersheetrefs" "${INTERSHEET_REFS}"
-			(at 447.9084 318.77 0)
+			(at 428.8584 299.72 0)
 			(effects
 				(font
@@
 			)
 		)
-		(property "Footprint" ""
+		(property "Footprint" "easyeda2kicad:Battery"
 			(at 182.88 150.876 90)
 			(effects
@@
 	(symbol
 		(lib_id "Connector:TestPoint")
-		(at 453.39 280.67 0)
+		(at 414.02 290.83 270)
 		(unit 1)
 		(exclude_from_sim no)
@@
 		(dnp no)
 		(property "Reference" "TP1"
-			(at 452.374 276.352 90)
+			(at 418.338 289.814 90)
 			(effects
 				(font
@@
 		)
 		(property "Value" "ADSB_CLK"
-			(at 454.152 276.352 90)
+			(at 418.338 291.592 90)
 			(effects
 				(font
@@
 		)
 		(property "Footprint" "easyeda2kicad:TestPoint"
-			(at 458.47 280.67 0)
+			(at 414.02 295.91 0)
 			(effects
 				(font
@@
 		)
 		(property "Datasheet" "~"
-			(at 458.47 280.67 0)
+			(at 414.02 295.91 0)
 			(effects
 				(font
@@
 		)
 		(property "Description" "test point"
-			(at 453.39 280.67 0)
+			(at 414.02 290.83 0)
 			(effects
 				(font

Commit message: checkpoint
Parts:
- BT1: now left out of the parts list
- C11, C12, C16, C17, C18, C19, C2, C20, C21, C22, C23, C24, C25, C26, C27, C30, C31, C32, C33, C34, C35, C36, C37, C38, C39, C40, C41, C42, C43, C44, C45, C46, C47, C48, C49, C50, C52, C54, C55, C56, C57, C58, C59, C60, C61, C62, C63, C64, C65, C66, C8, Card1, D2, D3, D4, J1, J2, L5, L6, L7, R1, R10, R11, R12, R14, R15, R16, R18, R19, R2, R20, R23, R24, R25, R28, R3, R30, R31, R32, R34, R35, R36, R37, R38, R39, R4, R40, R41, R44, R45, R46, R47, R5, R6, R7, R8, R9, SW1, SW2, SW4, SW5, U14, U19, USB1, USB2: now in the parts list
Connections:
- net BIAS_TEE_EN: now also U7.14 (GPIO11)
- net ADSB_CLK: now reaches TP1.1, U7.28 (GPIO17)
- net ADSB_CLK: now also U11.29 (IO34)
- no-connect marks 79 -> 78
Other:
- note added: "CH32V003 Power Control"
- note added: "ESP32S3 Main Processor"
- note added: "RP2040 CoProcessor"
- moved on the sheet: C18, C19, C20, C21, C22, C23, C24, C25, C26, C27, C28, C29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

Commit message: checkpoint
Parts:
- U11: LCSC Part (none) -> C22356044
- U7: LCSC Part (none) -> C2040
Changed lines of the file:
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@@
 			)
 		)
+		(property "LCSC Part" "C2040"
+			(at 308.61 281.94 0)
+			(effects
+				(font
+					(size 1.27 1.27)
+				)
+				(hide yes)
+			)
+		)
 		(pin "56"
 		)
@@
 			(effects
 				(font
+					(size 1.27 1.27)
+				)
+				(hide yes)
+			)
+		)
+		(property "LCSC Part" "C22356044"
+			(at 91.44 295.91 0)
+			(effects
+				(font
