File: PCB/RFlyOne.kicad_pcb (KiCad board)
At the start: 2 copper layers, 65 x 30 mm, 97 parts, among them J1 UFL, Q1 AO3401A, U1 TQP3M9036, U10 ATGM332D-5N31, U11 ESP32_S3_MINI, U12 E80-900M2212S, U13 RT9193-33GB, U14 RT8097CHGE, U15 BMI270, U16 MMC5983MA, U17 BQ25606RGER, U18 TPS61023DRLR, U19 CH32V003F4U6, U2 TLV3201, U3 TA0970A, U4 TQP3M9036, U5 TA0970A, U6 AD8313ARMZ, U7 RP2040, U8 W25Q128, U9 12MHz

Commit message: checkpoint
Parts:
- added C43: 1uF, Capacitor_SMD:C_0402_1005Metric, F.Cu at (58.3, 89.4)
- added C44: 47nF, Capacitor_SMD:C_0402_1005Metric, F.Cu at (58.3, 91.4)
- added C45: 10uF, Capacitor_SMD:C_0603_1608Metric, F.Cu at (67.6, 79.8)
- added C46: 10uF, Capacitor_SMD:C_0603_1608Metric, F.Cu at (67.6, 82.3)
- added C47: 4.7uF, Capacitor_SMD:C_0402_1005Metric, F.Cu at (58.3, 93.4)
- added C48: 10uF, Capacitor_SMD:C_0603_1608Metric, F.Cu at (67.6, 84.8)
- added C49: 10uF, Capacitor_SMD:C_0603_1608Metric, F.Cu at (67.6, 87.3)
- added C50: 10uF, Capacitor_SMD:C_0603_1608Metric, F.Cu at (67.6, 89.8)
- added C51: 22uF, Capacitor_SMD:C_0805_2012Metric, F.Cu at (71.8, 85.2)
- added C52: 0.1uF, Capacitor_SMD:C_0402_1005Metric, F.Cu at (61.1, 89.4)
- added C53: 22uF, Capacitor_SMD:C_0805_2012Metric, F.Cu at (71.8, 88.2)
- added C54: 0.1uF, Capacitor_SMD:C_0402_1005Metric, F.Cu at (61.1, 91.4)
- added C55: 0.1uF, Capacitor_SMD:C_0402_1005Metric, F.Cu at (61.1, 93.4)
- added C56: 0.1uF, Capacitor_SMD:C_0402_1005Metric, F.Cu at (64.0, 89.4)
- added C57: 0.1uF, Capacitor_SMD:C_0402_1005Metric, F.Cu at (64.0, 91.4)
- added C58: 1uF, Capacitor_SMD:C_0402_1005Metric, F.Cu at (64.0, 93.4)
- added C59: 1uF, Capacitor_SMD:C_0402_1005Metric, F.Cu at (55.4, 95.7)
- added J2: UFL, easyeda2kicad:UFL, F.Cu at (68.1, 93.6)
- added L6: 1.5uH, Inductor_SMD:L_Changjiang_FTC201610S, F.Cu at (72.4, 92.7)
- added L7: 1.5uH, Inductor_SMD:L_Changjiang_FTC201610S, F.Cu at (72.4, 96.1)
- added L8: 77nH, Inductor_SMD:L_0402_1005Metric, F.Cu at (58.3, 79.5)
- added Q2: AO3401A, Package_TO_SOT_SMD:SOT-23, F.Cu at (59.3, 96.6)
- added R23: 10k, Resistor_SMD:R_0402_1005Metric, F.Cu at (58.3, 81.5)
- added R24: 10k, Resistor_SMD:R_0402_1005Metric, F.Cu at (58.3, 83.5)
- added R25: 10k, Resistor_SMD:R_0402_1005Metric, F.Cu at (58.3, 85.5)
- added R26: 160R, Resistor_SMD:R_0402_1005Metric, F.Cu at (58.3, 87.5)
- added R27: 330R, Resistor_SMD:R_0402_1005Metric, F.Cu at (61.2, 79.5)
- added R28: 10k, Resistor_SMD:R_0402_1005Metric, F.Cu at (61.2, 81.5)
- added R29: 73.2k, Resistor_SMD:R_0402_1005Metric, F.Cu at (61.2, 83.5)
- added R30: 10k, Resistor_SMD:R_0402_1005Metric, F.Cu at (61.2, 85.5)
- added R31: 10k, Resistor_SMD:R_0402_1005Metric, F.Cu at (61.2, 87.5)
- added R32: 10k, Resistor_SMD:R_0402_1005Metric, F.Cu at (64.1, 79.5)
- added R33: 160R, Resistor_SMD:R_0402_1005Metric, F.Cu at (64.1, 81.5)
- added R34: 10k, Resistor_SMD:R_0402_1005Metric, F.Cu at (64.1, 83.5)
- added SW1: TS24CA, easyeda2kicad:SW-SMD_2P-TS24CA, F.Cu at (72.8, 81.6)
- added U20: TXU0202DTTR, easyeda2kicad:XSON-8_L2.0-W1.0-P0.50-BL, F.Cu at (63.6, 95.5)
- added U21: TPS7A0230-3V0, easyeda2kicad:SOT-23-5_L2.9-W1.6-P0.95-LS2.8-BR, F.Cu at (67.7, 98.1)
Connections:
- D2 pad 5: +5V -> +5VU
- D3 pad 5: +5V -> +5VU
- U10 pad 10: unconnected-(U10-GND-Pad10) -> GND
- U10 pad 11: unconnected-(U10-RF_IN-Pad11) -> Net-(J2-In)
- U10 pad 12: unconnected-(U10-GND-Pad12) -> GND
- U10 pad 13: unconnected-(U10-GND-Pad13) -> GND
- U10 pad 20: unconnected-(U10-TXD1-Pad20) -> GNSS_TX
- U10 pad 21: unconnected-(U10-RXD1-Pad21) -> GNSS_RX
- U10 pad 22: unconnected-(U10-VBAT-Pad22) -> +3V0
- U10 pad 23: unconnected-(U10-VCC-Pad23) -> +D3V3
- U10 pad 24: unconnected-(U10-GND-Pad24) -> GND
- U10 pad 3: unconnected-(U10-1PPS-Pad3) -> PPS
- U10 pad 9: unconnected-(U10-VCC_RF-Pad9) -> Net-(U10-VCC_RF)
- U17 pad 1: unconnected-(U17-VAC-Pad1) -> +5VU
- U17 pad 10: unconnected-(U17-ICHG-Pad10) -> Net-(U17-ICHG)
- U17 pad 11: unconnected-(U17-TS-Pad11) -> TS
- U17 pad 13: unconnected-(U17-BAT-Pad13) -> Net-(BT1-+)
- U17 pad 14: unconnected-(U17-BAT-Pad14) -> Net-(BT1-+)
- U17 pad 15: unconnected-(U17-SYS-Pad15) -> SYSTEM
- U17 pad 16: unconnected-(U17-SYS-Pad16) -> SYSTEM
- U17 pad 17: unconnected-(U17-GND-Pad17) -> GND
- U17 pad 18: unconnected-(U17-GND-Pad18) -> GND
- U17 pad 19: unconnected-(U17-SW-Pad19) -> Net-(C44-Pad2)
- U17 pad 20: unconnected-(U17-SW-Pad20) -> Net-(C44-Pad2)
- U17 pad 21: unconnected-(U17-BTST-Pad21) -> Net-(U17-BTST)
- U17 pad 22: unconnected-(U17-REGN-Pad22) -> REGN
- U17 pad 23: unconnected-(U17-PMID-Pad23) -> PMID
- U17 pad 24: unconnected-(U17-VBUS-Pad24) -> +5VU
- U17 pad 25: unconnected-(U17-EP-Pad25) -> GND
- U17 pad 5: unconnected-(U17-STAT-Pad5) -> CHARGE
- U17 pad 6: unconnected-(U17-OTG-Pad6) -> GND
- U17 pad 7: unconnected-(U17-~{PG}-Pad7) -> PG
- U17 pad 8: unconnected-(U17-ILIM-Pad8) -> Net-(U17-ILIM)
- U17 pad 9: unconnected-(U17-~{CE}-Pad9) -> CE
- U18 pad 1: unconnected-(U18-FB-Pad1) -> BOOST_FB
- U18 pad 2: unconnected-(U18-EN-Pad2) -> +BATT
- U18 pad 3: unconnected-(U18-VIN-Pad3) -> +BATT
- U18 pad 4: unconnected-(U18-GND-Pad4) -> GND
- U18 pad 5: unconnected-(U18-SW-Pad5) -> Net-(U18-SW)
- U18 pad 6: unconnected-(U18-VOUT-Pad6) -> +5V
- U19 pad 10: unconnected-(U19-PC3-Pad10) -> CHARGE
- U19 pad 15: unconnected-(U19-PD1-Pad15) -> Net-(U19-PD1)
- U19 pad 21: unconnected-(U19-VSS-Pad21) -> GND
- U19 pad 4: unconnected-(U19-VSS-Pad4) -> GND
- U19 pad 6: unconnected-(U19-VDD-Pad6) -> SYSTEM
- U19 pad 8: unconnected-(U19-PC1-Pad8) -> Net-(U19-PC1)
- U19 pad 9: unconnected-(U19-PC2-Pad9) -> PG
- USB1 pad 11: +5V -> +5VU
- USB1 pad 2: +5V -> +5VU
- USB2 pad 11: +5V -> +5VU
- USB2 pad 2: +5V -> +5VU

Commit message: checkpoint
Parts:
- added C60: 0.1uF, Capacitor_SMD:C_0402_1005Metric, F.Cu at (180.1, 102.3)
- added C61: 10uF, Capacitor_SMD:C_0603_1608Metric, F.Cu at (198.4, 98.8)
- added C62: 0.1uF, Capacitor_SMD:C_0402_1005Metric, F.Cu at (180.1, 104.2)
- added C63: 0.1uF, Capacitor_SMD:C_0402_1005Metric, F.Cu at (180.1, 106.2)
- added R35: 10k, Resistor_SMD:R_0402_1005Metric, F.Cu at (180.2, 116.2)
- added R36: 10k, Resistor_SMD:R_0402_1005Metric, F.Cu at (180.2, 118.1)
- added R37: 10k, Resistor_SMD:R_0402_1005Metric, F.Cu at (180.2, 120.1)
- added R38: 10k, Resistor_SMD:R_0402_1005Metric, F.Cu at (180.2, 122.1)
- added R39: 10k, Resistor_SMD:R_0402_1005Metric, F.Cu at (180.2, 124.1)
- added R40: 10k, Resistor_SMD:R_0402_1005Metric, F.Cu at (183.2, 108.2)
- added R41: 10k, Resistor_SMD:R_0402_1005Metric, F.Cu at (183.2, 110.2)
- added R42: 2.7k, Resistor_SMD:R_0402_1005Metric, F.Cu at (183.2, 112.2)
- added R43: 7.5k, Resistor_SMD:R_0402_1005Metric, F.Cu at (183.2, 114.2)
- added R44: 10k, Resistor_SMD:R_0402_1005Metric, F.Cu at (183.2, 116.2)
- added R45: 10k, Resistor_SMD:R_0402_1005Metric, F.Cu at (183.2, 118.1)
- added SW2: TS24CA, easyeda2kicad:SW-SMD_2P-TS24CA, F.Cu at (190.7, 68.5)
- added SW4: TS24CA, easyeda2kicad:SW-SMD_2P-TS24CA, F.Cu at (190.7, 73.6)
- added SW5: TS24CA, easyeda2kicad:SW-SMD_2P-TS24CA, F.Cu at (190.7, 78.8)
- added U22: 240x320_2.4in_TFT, easyeda2kicad:2.4TFT, F.Cu at (133.1, 55.0)
- U10, U11, U12: moved to F.Cu
- moved Q2 146.1 mm to (204.4, 113.9)
- moved U20 144.3 mm to (204.1, 128.2)
- moved L6 132.8 mm to (202.4, 65.3)
- moved L7 132.8 mm to (202.4, 68.6)
- moved C51 131.9 mm to (202.6, 102.1)
- moved C53 131.9 mm to (202.6, 105.1)
- moved C46 130.9 mm to (198.4, 88.8)
- moved C48 130.9 mm to (198.4, 91.3)
- moved C49 130.9 mm to (198.4, 93.8)
- moved C50 130.9 mm to (198.4, 96.3)
- moved C45 128.6 mm to (194.3, 101.3)
- moved C59 124.8 mm to (180.1, 100.3)
- moved R23 122.5 mm to (177.3, 110.2)
- moved R24 122.5 mm to (177.3, 112.2)
- moved R25 122.5 mm to (177.3, 114.2)
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Connections:
- net ESP32_RX renamed BTMGR_ESP32_RX
- net ESP32_TX renamed BTMGR_ESP32_TX
- Card1 pad 1: unconnected-(Card1-DATA2-Pad1) -> SDIO_DAT2
- Card1 pad 10: unconnected-(Card1-GND-Pad10) -> GND
- Card1 pad 11: unconnected-(Card1-GND-Pad11) -> GND
- Card1 pad 12: unconnected-(Card1-GND-Pad12) -> GND
- Card1 pad 13: unconnected-(Card1-GND-Pad13) -> GND
- Card1 pad 2: unconnected-(Card1-CD/DATA3-Pad2) -> SDIO_DAT3
- Card1 pad 3: unconnected-(Card1-CMD-Pad3) -> SDIO_CMD
- Card1 pad 4: unconnected-(Card1-VDD-Pad4) -> +D3V3
- Card1 pad 5: unconnected-(Card1-CLK-Pad5) -> SDIO_CLK
- Card1 pad 6: unconnected-(Card1-VSS-Pad6) -> GND
- Card1 pad 7: unconnected-(Card1-DAT0-Pad7) -> SDIO_DAT0
- Card1 pad 8: unconnected-(Card1-DAT1-Pad8) -> SDIO_DAT1
- Card1 pad 9: unconnected-(Card1-CD-Pad9) -> SDIO_CD
- R22 pad 1: unconnected-(R22-Pad1) -> SDA
- R22 pad 2: unconnected-(R22-Pad2) -> +D3V3
- R30 pad 1: CHARGE -> PG
- R31 pad 1: PG -> CHARGE
- SW1 pad 1: unconnected-(SW1-Pad1) -> PWR_BTN
- SW1 pad 2: unconnected-(SW1-Pad2) -> GND
- SW1 pad 3: unconnected-(SW1-Pad3) -> GND
- SW1 pad 4: unconnected-(SW1-Pad4) -> GND
- U11 pad 45: unconnected-(U11-EN-Pad45) -> Net-(U11-EN)
- U12 pad 1: unconnected-(U12-GND-Pad1) -> GND
- U12 pad 11: unconnected-(U12-GND-Pad11) -> GND
- U12 pad 13: unconnected-(U12-GND-Pad13) -> GND
- U12 pad 14: unconnected-(U12-GND-Pad14) -> GND
- U12 pad 16: unconnected-(U12-GND-Pad16) -> GND
- U12 pad 19: unconnected-(U12-GND-Pad19) -> GND
- U12 pad 21: unconnected-(U12-LR_NRESET-Pad21) -> Net-(U12-LR_NRESET)
- U12 pad 25: unconnected-(U12-VCC-Pad25) -> +D3V3
- U12 pad 26: unconnected-(U12-GND-Pad26) -> GND
- U12 pad 3: unconnected-(U12-MISO-Pad3) -> LORA_MISO
- U12 pad 4: unconnected-(U12-MOSI-Pad4) -> LORA_MOSI
- U12 pad 5: unconnected-(U12-SCK-Pad5) -> LORA_SCK
- U12 pad 6: unconnected-(U12-NSS-Pad6) -> LORA_CE
- U12 pad 7: unconnected-(U12-BUSY-Pad7) -> LORA_BUSY
- U12 pad 8: unconnected-(U12-GND-Pad8) -> GND
- U19 pad 10: CHARGE -> unconnected-(U19-PC3-Pad10)
- U19 pad 9: PG -> unconnected-(U19-PC2-Pad9)
- U7 pad 27: ESP_UART_TX -> unconnected-(U7-GPIO16-Pad27)
- U7 pad 28: ESP_UART_RX -> unconnected-(U7-GPIO17-Pad28)
- U7 pad 29: BIAS_TEE_EN -> unconnected-(U7-GPIO18-Pad29)
- U7 pad 30: PULSE -> unconnected-(U7-GPIO19-Pad30)
- U7 pad 36: Net-(U7-GPIO24) -> unconnected-(U7-GPIO24-Pad36)
- U7 pad 6: Net-(U7-GPIO4) -> unconnected-(U7-GPIO4-Pad6)
- U7 pad 7: Net-(U7-GPIO5) -> unconnected-(U7-GPIO5-Pad7)
Other:
- board size 65 x 30 mm -> 46 x 80 mm

Commit message: checkpoint
Parts:
- added R46: 10k, Resistor_SMD:R_0402_1005Metric, B.Cu at (155.1, 96.0)
- R10, R15, R18, R19, U12, U15: moved to B.Cu
- U11: footprint RF_Module:ESP32-S2-MINI-1U -> easyeda2kicad:ESP32-S2-MINI-1U; moved to B.Cu
- moved D3 65.6 mm to (142.3, 119.6)
- moved U15 59.1 mm to (131.6, 91.3), turned to 180 degrees
- moved U11 53.4 mm to (148.4, 87.1), turned to 90 degrees
- moved R15 49.6 mm to (127.1, 127.1), turned to -90 degrees
- moved R39 47.5 mm to (139.7, 99.3), turned to 180 degrees
- moved R38 47.1 mm to (139.7, 98.2), turned to 180 degrees
- moved R10 47.0 mm to (125.2, 128.6), turned to 180 degrees
- moved R37 46.6 mm to (139.7, 97.1), turned to 180 degrees
- moved R40 43.5 mm to (139.7, 105.9), turned to 180 degrees
- moved R36 42.7 mm to (139.7, 104.8), turned to 180 degrees
- moved R35 42.4 mm to (139.7, 103.7), turned to 180 degrees
- moved R18 33.1 mm to (142.1, 125.1), turned to -90 degrees
- moved R19 31.7 mm to (143.2, 125.1), turned to -90 degrees
- moved U12 25.1 mm to (147.6, 110.1), turned to 180 degrees
- moved USB2 16.2 mm to (142.3, 125.7)
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Connections:
- net CONN_RP_USB_DM renamed CONN_RP_USB_DN
- net RP_USB_DM renamed RP_USB_DN
- D3 pad 1: CONN_ESP_USB_DP -> CONN_ESP_USB_DN
- D3 pad 3: CONN_ESP_USB_DM -> CONN_ESP_USB_DP
- D3 pad 4: ESP_USB_DM -> ESP_USB_DP
- D3 pad 6: ESP_USB_DP -> ESP_USB_DN
- U11 pad 10: unconnected-(U11-IO6-Pad10) -> SDIO_CD
- U11 pad 11: unconnected-(U11-IO7-Pad11) -> SDIO_DAT1
- U11 pad 12: unconnected-(U11-IO8-Pad12) -> SDIO_DAT0
- U11 pad 13: unconnected-(U11-IO9-Pad13) -> SDIO_CLK
- U11 pad 14: unconnected-(U11-IO10-Pad14) -> SDIO_CMD
- U11 pad 15: unconnected-(U11-IO11-Pad15) -> SDIO_DAT3
- U11 pad 16: unconnected-(U11-IO12-Pad16) -> SDIO_DAT2
- U11 pad 23: ESP_USB_DM -> ESP_USB_DN
- U11 pad 4: unconnected-(U11-IO0-Pad4) -> Net-(U11-IO0)
- U11 pad 5: unconnected-(U11-IO1-Pad5) -> LORA_MISO
- U11 pad 6: unconnected-(U11-IO2-Pad6) -> LORA_MOSI
- U11 pad 7: unconnected-(U11-IO3-Pad7) -> LORA_SCK
- U11 pad 8: unconnected-(U11-IO4-Pad8) -> LORA_CE
- U11 pad 9: unconnected-(U11-IO5-Pad9) -> LORA_BUSY
- USB2 pad 5: CONN_ESP_USB_DM -> CONN_ESP_USB_DN
- USB2 pad 7: CONN_ESP_USB_DM -> CONN_ESP_USB_DN
Routing:
- net ESP_USB_DP: track 0.00 -> 34.7 mm, vias 0 -> 2
- net ESP_USB_DN: track 0.00 -> 34.6 mm, vias 0 -> 2
- net +5VU: track 0.00 -> 29.7 mm
- net LORA_BUSY: track 0.00 -> 16.5 mm
- net SDIO_CD: track 0.00 -> 15.7 mm, vias 0 -> 1
- net LORA_CE: track 0.00 -> 14.9 mm
- net SDIO_DAT1: track 0.00 -> 14.3 mm, vias 0 -> 1
- net LORA_SCK: track 0.00 -> 12.9 mm
- net SDIO_DAT0: track 0.00 -> 12.8 mm, vias 0 -> 1
- net LORA_MOSI: track 0.00 -> 11.3 mm
- net LORA_MISO: track 0.00 -> 9.61 mm
- net SDIO_CLK: track 0.00 -> 8.22 mm, vias 0 -> 1
- net SDIO_CMD: track 0.00 -> 7.70 mm, vias 0 -> 1
- net SDIO_DAT2: track 0.00 -> 7.44 mm, vias 0 -> 1
- net SDIO_DAT3: track 0.00 -> 6.44 mm, vias 0 -> 1
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- added copper zone on B.Cu, net GND
- added copper zone on F.Cu, net GND
- added copper zone on In1.Cu, net GND
- added copper zone on In2.Cu, net GND
Other:
- copper layers 2 -> 4

Commit message: checkpoint
Parts:
- added TP1: ADSB_CLK, easyeda2kicad:TestPoint, B.Cu at (163.7, 87.4)
- added TP10: ESP_RST, easyeda2kicad:TestPoint, B.Cu at (153.2, 78.3)
- added TP11: ESP_BOOT, easyeda2kicad:TestPoint, B.Cu at (151.9, 96.0)
- added TP2: SWCLK, easyeda2kicad:TestPoint, B.Cu at (163.7, 89.4)
- added TP3: SWDIO, easyeda2kicad:TestPoint, B.Cu at (163.7, 91.4)
- added TP4: BOOT, easyeda2kicad:TestPoint, B.Cu at (163.7, 93.4)
- added TP5: UART_TX, easyeda2kicad:TestPoint, B.Cu at (161.7, 87.4)
- added TP6: UART_RX, easyeda2kicad:TestPoint, B.Cu at (161.7, 89.4)
- added TP7: ESP_UART_RX, easyeda2kicad:TestPoint, B.Cu at (161.7, 91.4)
- added TP8: ESP_UART_TX, easyeda2kicad:TestPoint, B.Cu at (161.7, 93.4)
- added TP9: CH32_SWDIO, easyeda2kicad:TestPoint, B.Cu at (159.7, 87.4)
- C1, C10, C11, C12, C2, C3, C33, C34, C35, C37, C38, C39, C4, C40, C41, C42, C43, C44, C45, C46, C47, C48, C49, C5, C50, C51, C53, C57, C58, C59, C6, C61, C62, C7, C8, C9, D1, F1, J1, J2, L1, L2, L3, L4, L8, Q1, R1, R2, R20, R21, R22, R23, R24, R25, R26, R27, R28, R29, R3, R42, R45, U1, U10, U14, U16, U17, U18, U19, U2, U21, U3, U4, U5, U6: moved to B.Cu
- L5, L6, L7: footprint Inductor_SMD:L_Changjiang_FTC201610S -> easyeda2kicad:L_Changjiang_FTC201610S; moved to B.Cu
- moved D1 115.5 mm to (93.1, 97.9), turned to -90 degrees
- moved U6 110.6 mm to (93.6, 112.9)
- moved U5 107.7 mm to (97.5, 106.6), turned to -90 degrees
- moved Q1 107.3 mm to (97.6, 99.5), turned to 180 degrees
- moved L6 97.0 mm to (117.8, 112.8), turned to 180 degrees
- moved U3 96.6 mm to (102.6, 103.5), turned to 90 degrees
- moved U1 95.1 mm to (96.0, 103.3), turned to 90 degrees
- moved U4 93.3 mm to (104.0, 106.8), turned to -90 degrees
- moved L5 91.5 mm to (133.0, 121.6)
- moved L7 90.8 mm to (126.4, 118.4), turned to 90 degrees
- moved C46 86.4 mm to (117.3, 118.7), turned to -90 degrees
- moved C11 82.4 mm to (92.0, 110.4), turned to 90 degrees
- moved C49 82.3 mm to (117.8, 110.8)
- moved D2 81.7 mm to (126.3, 118.3)
- moved C48 79.8 mm to (120.9, 110.6), turned to 180 degrees
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Connections:
- U11 pad 10: SDIO_CD -> LORA_BUSY
- U11 pad 11: SDIO_DAT1 -> SDIO_CD
- U11 pad 12: SDIO_DAT0 -> SDIO_DAT1
- U11 pad 13: SDIO_CLK -> SDIO_DAT0
- U11 pad 14: SDIO_CMD -> SDIO_CLK
- U11 pad 15: SDIO_DAT3 -> SDIO_CMD
- U11 pad 17: unconnected-(U11-IO13-Pad17) -> SDIO_DAT3
- U11 pad 18: unconnected-(U11-IO14-Pad18) -> GNSS_RX
- U11 pad 19: unconnected-(U11-IO15-Pad19) -> GNSS_TX
- U11 pad 20: unconnected-(U11-IO16-Pad20) -> PPS
- U11 pad 31: unconnected-(U11-IO35-Pad31) -> SCL
- U11 pad 32: unconnected-(U11-IO36-Pad32) -> SDA
- U11 pad 33: unconnected-(U11-IO37-Pad33) -> TOUCH_IRQ
- U11 pad 34: unconnected-(U11-IO38-Pad34) -> TOUCH_CS
- U11 pad 35: unconnected-(U11-IO39-Pad35) -> LCD_MISO
- U11 pad 36: unconnected-(U11-IO40-Pad36) -> LCD_LED
- U11 pad 37: unconnected-(U11-IO41-Pad37) -> LCD_SCK
- U11 pad 38: unconnected-(U11-IO42-Pad38) -> LCD_MOSI
- U11 pad 39: unconnected-(U11-TXD0-Pad39) -> LCD_CMD
- U11 pad 40: unconnected-(U11-RXD0-Pad40) -> LCD_CS
- U11 pad 7: LORA_SCK -> unconnected-(U11-IO3-Pad7)
- U11 pad 8: LORA_CE -> LORA_SCK
- U11 pad 9: LORA_BUSY -> LORA_CE
Routing:
- net LCD_MOSI: track 0.00 -> 46.6 mm
- net +5VU: track 29.7 -> 75.4 mm, vias 0 -> 6
- net LCD_MISO: track 0.00 -> 43.6 mm
- net TOUCH_IRQ: track 0.00 -> 43.3 mm
- net LCD_SCK: track 0.00 -> 39.7 mm
- net TOUCH_CS: track 0.00 -> 36.2 mm
- net LCD_LED: track 0.00 -> 31.7 mm
- net LCD_CMD: track 0.00 -> 29.6 mm
- net LCD_CS: track 0.00 -> 27.8 mm
- net PPS: track 0.00 -> 21.8 mm, vias 0 -> 2
- net +D3V3: track 0.00 -> 16.9 mm
- net SCL: track 0.00 -> 15.3 mm, vias 0 -> 2
- net +5V: track 0.00 -> 14.3 mm
- net SDA: track 0.00 -> 12.6 mm
- net REGN: track 0.00 -> 12.4 mm, vias 0 -> 2
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
Commit message: checkpoint
Parts:
- added C64: 0.1uF, Capacitor_SMD:C_0402_1005Metric, F.Cu at (127.0, 78.3)
- added C65: 0.1uF, Capacitor_SMD:C_0402_1005Metric, F.Cu at (123.4, 78.1)
- added C66: 0.1uF, Capacitor_SMD:C_0402_1005Metric, F.Cu at (133.4, 70.9)
- C54, C55, C56, Q2, R30, R31, R32, R33, R34, R41, U20: moved to B.Cu
- TP4: value BOOT -> RP_BOOT
- moved SW2 80.0 mm to (112.7, 86.4), turned to 90 degrees
- moved SW5 79.7 mm to (112.7, 62.4), turned to 90 degrees
- moved SW4 78.0 mm to (112.7, 74.4), turned to 90 degrees
- moved U20 76.5 mm to (129.6, 111.1)
- moved U7 74.5 mm to (124.4, 72.7), turned to -90 degrees
- moved R12 72.6 mm to (128.3, 65.8), turned to 180 degrees
- moved R11 72.3 mm to (119.7, 71.7), turned to -90 degrees
- moved Q2 67.0 mm to (137.4, 114.1), turned to 90 degrees
- moved C28 66.2 mm to (117.5, 68.2), turned to 180 degrees
- moved R16 65.9 mm to (128.1, 67.3), turned to -90 degrees
- moved R14 65.5 mm to (119.2, 75.0), turned to 180 degrees
- moved U8 65.3 mm to (132.0, 65.6), turned to 180 degrees
- moved C29 64.6 mm to (119.7, 69.8), turned to -90 degrees
- moved C26 60.2 mm to (119.2, 74.1), turned to 180 degrees
- moved C24 59.1 mm to (119.2, 73.2), turned to 180 degrees
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Connections:
- net BTMGR_ESP32_RX renamed CONV_CH32_TX
- net BTMGR_ESP32_TX renamed CONV_CH32_RX
- D2 pad 1: CONN_RP_USB_DP -> CONN_RP_USB_DN
- D2 pad 3: CONN_RP_USB_DN -> CONN_RP_USB_DP
- D2 pad 4: RP_USB_DN -> RP_USB_DP
- D2 pad 6: RP_USB_DP -> RP_USB_DN
- R12 pad 1: Net-(U8-~{CS}) -> SPI_CS
- R16 pad 1: SPI_CS -> Net-(R16-Pad1)
- R16 pad 2: Net-(U8-~{CS}) -> SPI_CS
- TP4 pad 1: Net-(U8-~{CS}) -> Net-(R16-Pad1)
- U11 pad 10: LORA_BUSY -> BATT_ADC
- U11 pad 20: PPS -> LORA_BUSY
- U11 pad 21: unconnected-(U11-IO17-Pad21) -> PPS
- U19 pad 10: unconnected-(U19-PC3-Pad10) -> PG
- U19 pad 16: unconnected-(U19-PD2-Pad16) -> LEFT_BTN
- U19 pad 17: unconnected-(U19-PD3-Pad17) -> OK_BTN
- U19 pad 18: unconnected-(U19-PD4-Pad18) -> RIGHT_BTN
- U19 pad 19: unconnected-(U19-PD5-Pad19) -> CH32_TX
- U19 pad 20: unconnected-(U19-PD6-Pad20) -> CH32_RX
- U19 pad 9: unconnected-(U19-PC2-Pad9) -> CHARGE
- U8 pad 1: Net-(U8-~{CS}) -> SPI_CS
Routing:
- net PG: track 0.00 -> 24.4 mm, vias 0 -> 2
- net CHARGE: track 0.00 -> 22.6 mm, vias 0 -> 2
- net +D3V3: track 16.9 -> 34.0 mm
- net SPI_CS: track 0.00 -> 14.7 mm, vias 0 -> 2
- net SPI_SD2: track 0.00 -> 10.6 mm
- net SPI_SD1: track 0.00 -> 10.1 mm, vias 0 -> 2
- net LORA_BUSY: track 17.2 -> 24.3 mm, vias 0 -> 2
- net SYSTEM: track 12.4 -> 18.8 mm
- net SPI_SD3: track 0.00 -> 6.44 mm
- net GND: track 10.2 -> 15.9 mm, vias 20 -> 26
- net BATT_ADC: track 0.00 -> 5.01 mm, vias 0 -> 1
- net SPI_CLK: track 0.00 -> 5.01 mm
- net Net-(Q2-G): track 0.00 -> 4.98 mm
- net CONN_RP_USB_DP: track 0.00 -> 4.83 mm
- net Net-(U7-VREG_VOUT): track 0.00 -> 4.38 mm
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
Commit message: checkpoint
Parts:
- added TP12: D3V3, easyeda2kicad:TestPoint, B.Cu at (134.2, 124.5)
- added TP13: 3V3, easyeda2kicad:TestPoint, B.Cu at (125.3, 102.0)
- added TP14: 5V, easyeda2kicad:TestPoint, B.Cu at (127.0, 114.2)
- added TP15: 5VU, easyeda2kicad:TestPoint, B.Cu at (133.2, 127.1)
- added TP16: SDA, easyeda2kicad:TestPoint, B.Cu at (142.3, 73.2)
- added TP17: SCL, easyeda2kicad:TestPoint, B.Cu at (141.5, 78.1)
- added TP18: CHARGE, easyeda2kicad:TestPoint, B.Cu at (124.3, 116.5)
- added TP19: PG, easyeda2kicad:TestPoint, B.Cu at (123.8, 119.0)
- added TP20: PULSE, easyeda2kicad:TestPoint, B.Cu at (120.4, 101.8)
- C13, C14, C15, C16, C17, C30, C31, C32, C52, R4, R5, R6, R7, R8, R9, U13: moved to B.Cu
- moved R9 60.4 mm to (113.8, 100.5)
- moved C52 60.3 mm to (125.2, 113.4), turned to 180 degrees
- moved R6 58.1 mm to (114.2, 102.9), turned to 90 degrees
- moved C32 57.8 mm to (123.1, 110.8), turned to 90 degrees
- moved C17 57.7 mm to (113.8, 101.5)
- moved C14 57.5 mm to (114.9, 104.8), turned to -90 degrees
- moved R7 56.4 mm to (115.9, 104.8), turned to 90 degrees
- moved C31 55.7 mm to (125.5, 109.2)
- moved C16 55.7 mm to (115.8, 99.8), turned to 180 degrees
- moved R4 55.7 mm to (115.9, 106.7), turned to 90 degrees
- moved R8 55.5 mm to (116.8, 106.7), turned to -90 degrees
- moved C15 55.4 mm to (117.3, 108.1)
- moved R5 54.9 mm to (116.8, 104.8), turned to 90 degrees
- moved C13 54.4 mm to (118.3, 103.9)
- moved C30 49.8 mm to (125.2, 114.4), turned to 180 degrees
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Routing:
- net RIGHT_BTN: track 0.00 -> 58.6 mm, vias 0 -> 2
- net OK_BTN: track 0.00 -> 47.8 mm, vias 0 -> 2
- net LEFT_BTN: track 0.00 -> 36.3 mm, vias 0 -> 2
- net SYSTEM: track 18.8 -> 47.9 mm, vias 0 -> 4
- net +BATT: track 3.58 -> 21.6 mm, vias 0 -> 5
- net +5V: track 14.3 -> 25.1 mm
- net +3V3: track 0.00 -> 9.50 mm
- net +D3V3: track 34.0 -> 43.5 mm, vias 0 -> 4
- net Net-(U6-VOUT): track 0.00 -> 5.92 mm
- net Net-(U2-IN-): track 0.00 -> 4.16 mm
- net GND: track 15.9 -> 19.8 mm, vias 26 -> 133
- net +5VU: track 75.4 -> 78.7 mm
- net Net-(D1-A2): track 5.75 -> 2.87 mm
- net PULSE: track 0.00 -> 2.63 mm
- net Net-(U2-IN+): track 0.00 -> 2.37 mm
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Other:
- board text added: "+5V"
- board text added: "+5VU"
- board text added: "+D3V3"
- board text added: "ADSB_ANT"
- board text added: "ATGM332D"
- board text added: "BOOT"
- board text added: "CHRG"
- board text added: "E80-900M2212S"
- board text added: "ESP32"
- board text added: "ESP32S3"
- board text added: "GPS_ANT"
- board text added: "MicroSD"
- board text added: "PG"
- board text added: "PWR"
- board text added: "RP2040"
- board text added: "RP_BOOT"
- board text added: "RST"
- board text added: "SCL"
- board text added: "SDA"
- board text added: "SWCLK"
- board text added: "SWD"
- board text added: "SWDIO"
