File: PCB/RFlyOne.kicad_pcb (KiCad board)
At the start: 4 copper layers, 46 x 80 mm, 177 parts, among them J1 UFL, J2 UFL, Q1 AO3401A, Q2 AO3401A, SW1 TS24CA, SW2 TS24CA, SW4 TS24CA, SW5 TS24CA, U1 TQP3M9036, U10 ATGM332D-5N31, U11 ESP32_S3_MINI, U12 E80-900M2212S, U13 RT9193-33GB, U14 RT8097CHGE, U15 BMI270, U16 MMC5983MA, U17 BQ25606RGER, U18 TPS61023DRLR, U19 CH32V003F4U6, U2 TLV3201, U20 TXU0202DTTR, U21 TPS7A0230-3V0, U22 240x320_2.4in_TFT, U3 TA0970A, U4 TQP3M9036, U5 TA0970A, U6 AD8313ARMZ, U7 RP2040, U8 W25Q128, U9 12MHz

Commit message: checkpoint
Parts:
- added D4: WHITE, easyeda2kicad:LED-SMD_L1.6-W1.1-R-RD_WHITE, F.Cu at (156.4, 80.3)
- added JP1: ChargeDisable, Jumper:SolderJumper-2_P1.3mm_Open_RoundedPad1.0x1.5mm, F.Cu at (127.8, 85.7)
- added JP2: PWRBYPASS, Jumper:SolderJumper-2_P1.3mm_Open_RoundedPad1.0x1.5mm, F.Cu at (128.2, 89.0)
- added R47: 5.1k, Resistor_SMD:R_0402_1005Metric, F.Cu at (154.7, 82.0)
- added TP21: CH32_TX, easyeda2kicad:TestPoint, B.Cu at (135.2, 108.8)
- added TP22: CH32_RX, easyeda2kicad:TestPoint, B.Cu at (135.7, 105.6)
- TP5: value UART_TX -> RP_TX
- TP6: value UART_RX -> RP_RX
- moved TP8 24.8 mm to (138.9, 83.7)
- moved TP7 24.4 mm to (139.2, 82.1)
- moved C29 4.16 mm to (117.2, 73.2), turned to 0 degrees
- moved C64 0.18 mm to (127.0, 78.1)
- moved C23 0.07 mm to (123.5, 67.5)
Connections:
- TP5 pad 1: unconnected-(TP5-Pad1) -> Net-(U7-GPIO0)
- TP6 pad 1: unconnected-(TP6-Pad1) -> Net-(U7-GPIO1)
- TP7 pad 1: unconnected-(TP7-Pad1) -> RP2040_TX
- TP8 pad 1: unconnected-(TP8-Pad1) -> RP2040_RX
- U11 pad 22: unconnected-(U11-IO18-Pad22) -> CONV_CH32_RX
- U11 pad 25: unconnected-(U11-IO21-Pad25) -> CONV_CH32_TX
- U11 pad 27: unconnected-(U11-IO47-Pad27) -> RP2040_TX
- U11 pad 30: unconnected-(U11-IO48-Pad30) -> RP2040_RX
- U19 pad 2: unconnected-(U19-PA1-Pad2) -> Net-(U19-PA1)
- U19 pad 5: unconnected-(U19-PD0-Pad5) -> PWR_BTN
- U7 pad 2: unconnected-(U7-GPIO0-Pad2) -> Net-(U7-GPIO0)
- U7 pad 27: unconnected-(U7-GPIO16-Pad27) -> PULSE
- U7 pad 3: unconnected-(U7-GPIO1-Pad3) -> Net-(U7-GPIO1)
- U7 pad 6: unconnected-(U7-GPIO4-Pad6) -> RP2040_TX
- U7 pad 7: unconnected-(U7-GPIO5-Pad7) -> RP2040_RX
Routing:
- net +D3V3: track 43.5 -> 257.8 mm, vias 4 -> 17
- net PWR_BTN: track 0.00 -> 61.8 mm, vias 0 -> 1
- net Net-(U7-USB_DM): track 0.00 -> 53.6 mm, vias 0 -> 2
- net Net-(U7-USB_DP): track 0.00 -> 52.8 mm, vias 0 -> 2
- net +3V3: track 9.50 -> 59.8 mm, vias 0 -> 7
- net Net-(U19-PA1): track 0.00 -> 45.8 mm, vias 0 -> 1
- net GND: track 19.8 -> 61.5 mm, vias 133 -> 167
- net CONV_CH32_TX: track 0.00 -> 38.9 mm, vias 0 -> 3
- net CONV_CH32_RX: track 0.00 -> 35.7 mm, vias 0 -> 3
- net SYSTEM: track 47.9 -> 83.0 mm, vias 4 -> 5
- net +BATT: track 21.6 -> 51.5 mm, vias 5 -> 6
- net Net-(U7-VREG_VOUT): track 4.38 -> 17.1 mm, vias 0 -> 3
- net +5VU: track 78.7 -> 89.5 mm
- net Net-(U7-XIN): track 1.53 -> 7.41 mm
- net Net-(D4-A): track 0.00 -> 2.90 mm
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Other:
- board text added: "CH32_RX"
- board text added: "CH32_TX"

Commit message: checkpoint
Parts:
- added BT1: BAT, easyeda2kicad:Battery, B.Cu at (117.2, 122.5)
- added REF**: MountingHole, easyeda2kicad:MountingHole, F.Cu at (113.8, 53.1)
- added REF**: MountingHole, easyeda2kicad:MountingHole, F.Cu at (154.8, 53.1)
- added REF**: MountingHole, easyeda2kicad:MountingHole, F.Cu at (113.8, 128.1)
- added REF**: MountingHole, easyeda2kicad:MountingHole, F.Cu at (154.8, 128.1)
- moved TP6 45.2 mm to (123.3, 65.5), turned to 90 degrees
- moved TP5 41.8 mm to (126.0, 65.5), turned to 90 degrees
- moved TP1 40.9 mm to (124.7, 75.0)
- moved JP1 36.6 mm to (119.6, 121.3), turned to 180 degrees
- moved JP2 27.4 mm to (138.7, 114.3), turned to 90 degrees
- moved TP8 2.97 mm to (139.5, 80.8)
- moved TP7 1.62 mm to (139.5, 83.7)
- moved C46 0.67 mm to (116.6, 118.7)
Connections:
- TP1 pad 1: unconnected-(TP1-Pad1) -> Net-(U7-GPIO17)
- U7 pad 28: unconnected-(U7-GPIO17-Pad28) -> Net-(U7-GPIO17)
Routing:
- net RSSI: track 0.96 -> 40.5 mm, vias 0 -> 1
- net LEVEL_BIAS: track 1.88 -> 39.0 mm, vias 0 -> 1
- net +D3V3: track 257.8 -> 292.7 mm, vias 17 -> 21
- net PULSE: track 2.63 -> 33.5 mm
- net LEVEL_PWM: track 0.00 -> 30.0 mm, vias 0 -> 1
- net RP2040_RX: track 0.00 -> 27.3 mm, vias 0 -> 2
- net RP2040_TX: track 0.00 -> 27.0 mm, vias 0 -> 2
- net +3V3: track 59.8 -> 76.8 mm, vias 7 -> 8
- net GND: track 61.5 -> 69.5 mm, vias 167 -> 232
- net Net-(U7-GPIO1): track 0.00 -> 5.22 mm, vias 0 -> 1
- net Net-(BT1-+): track 4.99 -> 10.0 mm
- net Net-(U7-GPIO0): track 0.00 -> 4.02 mm, vias 0 -> 1
- net Net-(U7-GPIO17): track 0.00 -> 3.95 mm, vias 0 -> 1
- net CE: track 3.54 -> 5.60 mm, vias 0 -> 1
- net SCL: track 16.4 -> 17.5 mm
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Other:
- board text added: "+3V3"
- board text added: "ADSB_CLK"
- board text added: "ADSB_PPM"
- board text added: "CHRG DISAB"
- board text added: "DOWN"
- board text added: "PWR BYPASS"
- board text added: "RP_RX0"
- board text added: "RP_RX1"
- board text added: "RP_TX0"
- board text added: "RP_TX1"
- board text added: "SELECT"
- board text added: "UP"
