File: PCB/RFlyOne.kicad_pcb (KiCad board)
At the start: 4 copper layers, 46 x 80 mm, 188 parts, among them J1 UFL, J2 UFL, Q1 AO3401A, Q2 AO3401A, SW1 TS24CA, SW2 TS24CA, SW4 TS24CA, SW5 TS24CA, U1 TQP3M9036, U10 ATGM332D-5N31, U11 ESP32_S3_MINI, U12 E80-900M2212S, U13 RT9193-33GB, U14 RT8097CHGE, U15 BMI270, U16 MMC5983MA, U17 BQ25606RGER, U18 TPS61023DRLR, U19 CH32V003F4U6, U2 TLV3201, U20 TXU0202DTTR, U21 TPS7A0230-3V0, U22 240x320_2.4in_TFT, U3 TA0970A, U4 TQP3M9036, U5 TA0970A, U6 AD8313ARMZ, U7 RP2040, U8 W25Q128, U9 12MHz

Commit message: checkpoint
Connections:
- TP1 pad 1: Net-(U7-GPIO17) -> ADSB_CLK
- U11 pad 29: unconnected-(U11-IO34-Pad29) -> ADSB_CLK
- U7 pad 14: unconnected-(U7-GPIO11-Pad14) -> BIAS_TEE_EN
- U7 pad 28: Net-(U7-GPIO17) -> ADSB_CLK
Routing:
- net BIAS_TEE_EN: track 1.62 -> 29.4 mm, vias 0 -> 1
- net ADSB_CLK: track 0.00 -> 24.7 mm, vias 0 -> 1
- net Net-(U7-GPIO17): track 3.95 -> 0.00 mm, vias 1 -> 0
- net GND: vias 232 -> 244
- net (no net): vias 0 -> 1
